File: uController PCB1.kicad_pcb (KiCad board)
At the start: 2 copper layers, 104 parts, among them CN1 USB, J2 JUMPER2, J3 JUMPER3, J4 JUMPER2, J51 Conn_01x06_Pin, P10 Conn_01x01_Pin, P11 Conn_01x01_Pin, P12 Conn_01x01_Pin, P13 Conn_01x01_Pin, P14 Conn_01x01_Pin, P15 Conn_01x01_Pin, P16 Conn_01x01_Pin, P17 Conn_01x01_Pin, P2 Conn_01x01_Pin, P3 Conn_01x01_Pin, P4 Conn_01x01_Pin, P5 Conn_01x01_Pin, P6 Conn_01x01_Pin, P7 Conn_01x01_Pin, P8 Conn_01x01_Pin, P9 Conn_01x01_Pin, SW1 SW KEY-SPST, U1 FT231XS, U2 PIC18F4550-IP, U3 LD1117S33TR_SOT223, U4 CXO_DIP8

Commit message: Add files via upload
Parts:
- removed C1: 0.1uF, Capacitor_THT:C_Radial_D5.0mm_H5.0mm_P2.00mm
- removed CN1: USB, Package_DFN_QFN:WDFN-10-1EP_3x3mm_P0.5mm_EP1.8x2.5mm
- added C22: 0.1uF, Capacitor_SMD:C_0603_1608Metric, F.Cu at (237.9, 121.2)
- added C23: 0.1uF, Capacitor_SMD:C_0603_1608Metric, F.Cu at (237.9, 123.7)
- added C24: 10uF, Capacitor_SMD:C_1206_3216Metric, F.Cu at (250.7, 132.7)
- added C25: 47pF, Capacitor_SMD:C_0603_1608Metric, F.Cu at (237.9, 126.2)
- added C26: 0.1uF, Capacitor_SMD:C_0603_1608Metric, F.Cu at (237.9, 128.7)
- added C27: 47pF, Capacitor_SMD:C_0603_1608Metric, F.Cu at (237.9, 131.2)
- added C28: 0.1uF, Capacitor_SMD:C_0603_1608Metric, F.Cu at (237.9, 133.8)
- added C29: 0.1uF, Capacitor_SMD:C_0603_1608Metric, F.Cu at (241.9, 121.2)
- added C30: 0.1uF, Capacitor_SMD:C_0603_1608Metric, F.Cu at (241.9, 123.7)
- added D5: LED, LED_SMD:LED_0805_2012Metric, F.Cu at (233.1, 126.6)
- added D6: LED, LED_SMD:LED_0805_2012Metric, F.Cu at (233.1, 129.6)
- added J1: SCREWTERM, TestPoint:TestPoint_Bridge_Pitch3.81mm_Drill1.3mm, F.Cu at (114.7, 30.5)
- added J5: USB_B, Connector_USB:USB_B_TE_5787834_Vertical, F.Cu at (142.5, 22.5)
- added L2: FerriteBead, Inductor_SMD:L_0805_2012Metric, F.Cu at (233.1, 132.5)
- added P20: Conn_01x01_Pin, TestPoint:TestPoint_Loop_D2.54mm_Drill1.5mm_Beaded, F.Cu at (233.3, 107.4)
- added P21: Conn_01x01_Pin, TestPoint:TestPoint_Loop_D2.54mm_Drill1.5mm_Beaded, F.Cu at (233.3, 112.5)
- added P22: Conn_01x01_Pin, TestPoint:TestPoint_Loop_D2.54mm_Drill1.5mm_Beaded, F.Cu at (233.3, 117.5)
- added P23: Conn_01x01_Pin, TestPoint:TestPoint_Loop_D2.54mm_Drill1.5mm_Beaded, F.Cu at (233.3, 122.5)
- added R14: 27, Resistor_SMD:R_0603_1608Metric, F.Cu at (241.9, 131.2)
- added R15: 10k, Resistor_SMD:R_0603_1608Metric, F.Cu at (241.9, 133.8)
- added R16: 27, Resistor_SMD:R_0603_1608Metric, F.Cu at (245.9, 121.2)
- added R17: 180, Resistor_SMD:R_0603_1608Metric, F.Cu at (245.9, 123.7)
- added R18: 180, Resistor_SMD:R_0603_1608Metric, F.Cu at (245.9, 126.2)
- added R7: 10k, Resistor_SMD:R_0603_1608Metric, F.Cu at (106.0, 62.5)
- added R9: 10K, Resistor_SMD:R_0603_1608Metric, F.Cu at (117.2, 140.5)
- added RV1: R_Potentiometer, Potentiometer_THT:Potentiometer_Bourns_3386P_Vertical, F.Cu at (206.0, 86.1)
- C10: footprint Capacitor_THT:C_Radial_D5.0mm_H5.0mm_P2.00mm -> Capacitor_SMD:CP_Elec_5x5.4
- C9: footprint Capacitor_THT:C_Radial_D5.0mm_H5.0mm_P2.00mm -> Capacitor_THT:CP_Radial_D6.3mm_P2.50mm
- J2, J4: footprint Jumper:SolderJumper-2_P1.3mm_Bridged2Bar_Pad1.0x1.5mm -> TestPoint:TestPoint_Bridge_Pitch3.81mm_Drill1.3mm
- J3: footprint Jumper:SolderJumper-3_P1.3mm_Bridged2Bar12_Pad1.0x1.5mm -> Jumper:SolderJumper-3_P1.3mm_Open_Pad1.0x1.5mm
- J51: footprint LED_THT:LED_D5.0mm_IRGrey -> TestPoint:TestPoint_Loop_D2.54mm_Drill1.5mm_Beaded
- P11, P12, P13, P14, P15, P16, P17, P18, P19, P2, P3, P4, P5, P6, TP1, TP10, TP11, TP12, TP13, TP14, TP15, TP16, TP17, TP18, TP19, TP2, TP20, TP21, TP22, TP23, TP24, TP25, TP3, TP4, TP5, TP6, TP7, TP9: footprint Inductor_SMD:L_0805_2012Metric -> TestPoint:TestPoint_Loop_D2.54mm_Drill1.5mm_Beaded
- R10, R13, R8: footprint Resistor_SMD:R_0201_0603Metric -> Resistor_SMD:R_0603_1608Metric
- R11, R12: footprint Resistor_SMD:R_0508_1220Metric -> Resistor_THT:R_Axial_DIN0207_L6.3mm_D2.5mm_P10.16mm_Horizontal
- SW1: footprint Button_Switch_SMD:SW_Tactile_SPST_NO_Straight_CK_PTS636Sx25SMTRLFS -> Button_Switch_THT:SW_PUSH-12mm
- TP26, TP27, TP28, TP30, TP31, TP32, TP33, TP34, TP35, TP61, TP81, TP91: footprint Module:Flipper_Zero_Angled -> TestPoint:TestPoint_Loop_D2.54mm_Drill1.5mm_Beaded
- U4: footprint Oscillator:Oscillator_DIP-8 -> Oscillator:Oscillator_DIP-8_LargePads
- moved FID2 254.6 mm to (250.5, 16.0)
- moved FID4 237.2 mm to (258.5, 158.0)
- moved J3 233.3 mm to (256.4, 138.0)
- moved SW1 188.8 mm to (160.5, 29.5)
- moved J51 168.5 mm to (166.5, 55.0)
- moved J4 154.5 mm to (200.2, 72.0)
- moved TP16 146.8 mm to (166.5, 81.5)
- moved R13 136.4 mm to (184.0, 132.5)
- moved FID1 133.1 mm to (88.0, 17.5)
- moved J2 131.5 mm to (131.0, 39.3), turned to 90 degrees
- moved U1 120.6 mm to (141.1, 50.9), turned to 90 degrees
- moved C10 108.0 mm to (117.0, 48.5), turned to 90 degrees
- moved C9 103.1 mm to (116.0, 40.0)
- moved TP91 94.2 mm to (125.5, 89.5)
- moved R4 90.7 mm to (228.7, 84.5)
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- renumbered U3 to U2, U2 to U3
Connections:
- J4 pad 1: unconnected-(J4-A-Pad1) -> Net-(J4-A)
- R11 pad 1: unconnected-(R11-Pad1) -> /SCL
- R11 pad 2: VCC -> GND
- R12 pad 1: unconnected-(R12-Pad1) -> /SDA
- R12 pad 2: VCC -> GND
- R8 pad 1: unconnected-(R8-Pad1) -> /RB3
- TP30 pad 1: Net-(U2-RB0/AN12/INT0/FLT0/SDI/SDA) -> /SDA
- TP31 pad 1: Net-(U2-RB1/AN10/INT1/SCK/SCL) -> /SCL
- TP33 pad 1: Net-(U2-RB3/AN9/CCP2/VPO) -> /RB3
- TP6 pad 1: /USB_RXD -> /RX
- TP7 pad 1: /USB_TXD -> /TX
- U3 pad 13: unconnected-(U2-OSC1/CLKI-Pad13) -> /clk
- U3 pad 25: /USB_RXD -> /RX
- U3 pad 26: /USB_TXD -> /TX
- U3 pad 33: Net-(U2-RB0/AN12/INT0/FLT0/SDI/SDA) -> /SDA
- U3 pad 34: Net-(U2-RB1/AN10/INT1/SCK/SCL) -> /SCL
- U3 pad 36: Net-(U2-RB3/AN9/CCP2/VPO) -> /RB3
- U4 pad 5: unconnected-(U4-OUT-Pad5) -> /clk
Routing:
- net Net-(CN1-D-): track 290.5 -> 0.00 mm
- net VCC: track 230.8 -> 2.69 mm
- net GND: track 130.7 -> 0.94 mm
- net Net-(U3-RA5/AN4/~{SS}/HLVDIN/C2OUT): track 73.9 -> 0.00 mm
- net (no net): track 69.5 -> 0.00 mm
- net Net-(P9-Pin_1): track 60.4 -> 0.00 mm
- net +3.3V: track 51.8 -> 0.00 mm
- net Net-(U1-USBDM): track 48.4 -> 0.00 mm
- net Net-(CN1-VBUS): track 41.4 -> 0.60 mm
- net Net-(U2-VI): track 35.9 -> 0.00 mm
- net Net-(J51-Pin_5): track 0.00 -> 19.4 mm
- net Net-(J4-B): track 17.6 -> 0.00 mm
- net /USB_TXD: track 16.5 -> 0.00 mm
- net Net-(U3-VUSB): track 10.1 -> 0.00 mm
- net Net-(J51-Pin_1): track 6.62 -> 16.6 mm
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